File: KiCad/Complete-Rover-Systems/Complete-Rover-Systems.kicad_sch (KiCad schematic)
At the start: 1 part

Commit message: updated rover with imu
Connections:
- net RotaryEncoderSystem/B0: now also A1.25 (A6); no longer A1.23 (SDA/A4)
- net IMU/SCL: now reaches A1.24 (SCL/A5)
- new net IMU/SDA: A1.23 (SDA/A4)
Other:
- added sheet IMU (IMU.kicad_sch)
Changed lines of the file:
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@@
 			(width 0)
 			(type default)
-			(color 255 0 0 1)
 		)
 	)
@@
 			(width 0)
 			(type default)
-			(color 1 0 0 1)
 		)
 	)
@@
 	(wire
 		(pts
+			(xy 149.86 69.85) (xy 149.86 66.04)
+		)
+		(stroke
+			(width 0)
+			(type default)
+		)
+	)
+	(wire
+		(pts
 			(xy 59.69 127) (xy 104.14 127)
 		)
@@
 			(width 0)
 			(type default)
-			(color 1 0 0 1)
 		)
 	)
@@
 	(wire
 		(pts
+			(xy 129.54 121.92) (xy 153.67 121.92)
+		)
+		(stroke
+			(width 0)
+			(type default)
+		)
+	)
+	(wire
+		(pts
 			(xy 59.69 114.3) (xy 71.12 114.3)
 		)
@@
 	(wire
 		(pts
+			(xy 153.67 121.92) (xy 153.67 66.04)
+		)
+		(stroke
+			(width 0)
+			(type default)
+		)
+	)
+	(wire
+		(pts
 			(xy 80.01 83.82) (xy 80.01 109.22)
 		)
@@
 			(width 0)
 			(type default)
-			(color 1 0 0 1)
 		)
 	)
@@
 	(wire
 		(pts
-			(xy 149.86 119.38) (xy 149.86 82.55)
+			(xy 149.86 124.46) (xy 149.86 82.55)
 		)
 		(stroke
@@
 	(wire
 		(pts
+			(xy 139.7 119.38) (xy 139.7 69.85)
+		)
+		(stroke
+			(width 0)
+			(type default)
+		)
+	)
+	(wire
+		(pts
 			(xy 104.14 106.68) (xy 102.87 106.68)
 		)
@@
 	(wire
 		(pts
+			(xy 129.54 119.38) (xy 139.7 119.38)
+		)
+		(stroke
+			(width 0)
+			(type default)
+		)
+	)
+	(wire
+		(pts
 			(xy 133.35 140.97) (xy 49.53 140.97)
 		)
@@
 			(width 0)
 			(type default)
-			(color 255 0 0 1)
 		)
 	)
@@
 			(width 0)
 			(type default)
-			(color 1 0 0 1)
 		)
 	)
@@
 			(width 0)
 			(type default)
-			(color 1 0 0 1)
 		)
 	)
@@
 			(width 0)
 			(type default)
-			(color 1 0 0 1)
 		)
 	)
@@
 			(width 0)
 			(type default)
-			(color 255 0 0 1)
 		)
 	)
@@
 			(width 0)
 			(type default)
-			(color 255 0 0 1)
 		)
 	)
@@
 	(wire
 		(pts
-			(xy 129.54 119.38) (xy 149.86 119.38)
+			(xy 129.54 124.46) (xy 149.86 124.46)
 		)
 		(stroke
@@
 			(width 0)
 			(type default)
-			(color 255 0 0 1)
 		)
 	)
@@
 			(width 0)
 			(type default)
-			(color 255 0 0 1)
 		)
 	)
@@
 			(width 0)
 			(type default)
-			(color 255 0 0 1)
 		)
 	)
@@
 			(width 0)
 			(type default)
-			(color 1 0 0 1)
 		)
 	)
@@
 		(pts
 			(xy 45.72 83.82) (xy 80.01 83.82)
+		)
+		(stroke
+			(width 0)
+			(type default)
+		)
+	)
+	(wire
+		(pts
+			(xy 139.7 69.85) (xy 149.86 69.85)
 		)
 		(stroke
@@
 				)
 			)
+		)
+	)
+	(sheet
+		(at 143.51 46.99)
+		(size 20.32 19.05)
+		(fields_autoplaced yes)
+		(stroke
+			(width 0.1524)
+			(type solid)
+		)
+		(fill
+			(color 0 0 0 0.0000)
+		)
+		(property "Sheetname" "IMU"
+			(at 143.51 46.2784 0)
+			(effects
+				(font
+					(size 1.27 1.27)
+				)
+				(justify left bottom)
+			)
+		)
+		(property "Sheetfile" "IMU.kicad_sch"
+			(at 143.51 66.6246 0)
+			(effects
+				(font
+					(size 1.27 1.27)
+				)
+				(justify left top)
+			)
+		)
+		(pin "GND" input
+			(at 163.83 50.8 0)
+			(effects
+				(font
+					(size 1.27 1.27)
+				)
+				(justify right)
+			)
+		)
+		(pin "Vin (3.3V)" input
+			(at 163.83 54.61 0)
+			(effects
+				(font
+					(size 1.27 1.27)
+				)
+				(justify right)
+			)
+		)
+		(pin "SCL" input
+			(at 153.67 66.04 270)
+			(effects
+				(font
+					(size 1.27 1.27)
+				)
+				(justify left)
+			)
+		)
+		(pin "SDA" bidirectional
+			(at 149.86 66.04 270)
+			(effects
+				(font
+					(size 1.27 1.27)
+				)
+				(justify left)
+			)
+		)
+		(instances
+			(project "Complete-Rover-Systems"
+				(path "/6fa62cff-8e96-404b-9f84-9cfa132ad8cc"
+					(page "10")
+				)
+			)

Commit message: updated kicads
Other:
- sheet PowerSystemRover ports: added Vout (5V); removed none
Changed lines of the file:
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@@
 	(paper "A4")
+	(junction
+		(at 154.94 158.75)
+		(diameter 0)
+		(color 0 0 0 0)
+	)
 	(junction
 		(at 144.78 156.21)
@@
 	)
 	(junction
-		(at 154.94 160.02)
+		(at 160.02 166.37)
 		(diameter 0)
 		(color 0 0 0 0)
 	)
 	(junction
-		(at 160.02 166.37)
+		(at 156.21 156.21)
 		(diameter 0)
 		(color 0 0 0 0)
@@
 	)
 	(junction
-		(at 156.21 156.21)
-		(diameter 0)
-		(color 0 0 0 0)
-	)
-	(junction
 		(at 76.2 166.37)
 		(diameter 0)
@@
 	(wire
 		(pts
+			(xy 154.94 158.75) (xy 154.94 160.02)
+		)
+		(stroke
+			(width 0)
+			(type default)
+		)
+	)
+	(wire
+		(pts
 			(xy 160.02 166.37) (xy 171.45 166.37)
 		)
@@
 	(wire
 		(pts
-			(xy 154.94 151.13) (xy 154.94 160.02)
+			(xy 154.94 151.13) (xy 154.94 158.75)
+		)
+		(stroke
+			(width 0)
+			(type default)
+		)
+	)
+	(wire
+		(pts
+			(xy 62.23 156.21) (xy 88.9 156.21)
 		)
 		(stroke
@@
 	(wire
 		(pts
-			(xy 45.72 95.25) (xy 74.93 95.25)
-		)
-		(stroke
-			(width 0)
-			(type default)
-		)
-	)
-	(wire
-		(pts
 			(xy 82.55 101.6) (xy 104.14 101.6)
 		)
@@
 	(wire
 		(pts
+			(xy 71.12 146.05) (xy 71.12 166.37)
+		)
+		(stroke
+			(width 0)
+			(type default)
+		)
+	)
+	(wire
+		(pts
 			(xy 100.33 92.71) (xy 100.33 91.44)
 		)
@@
 	(wire
 		(pts
-			(xy 74.93 156.21) (xy 88.9 156.21)
-		)
-		(stroke
-			(width 0)
-			(type default)
-		)
-	)
-	(wire
-		(pts
 			(xy 116.84 166.37) (xy 157.48 166.37)
 		)
@@
 	(wire
 		(pts
-			(xy 71.12 146.05) (xy 71.12 166.37)
-		)
-		(stroke
-			(width 0)
-			(type default)
-		)
-	)
-	(wire
-		(pts
 			(xy 62.23 166.37) (xy 71.12 166.37)
 		)
@@
 	(wire
 		(pts
-			(xy 74.93 95.25) (xy 74.93 156.21)
-		)
-		(stroke
-			(width 0)
-			(type default)
-		)
-	)
-	(wire
-		(pts
 			(xy 59.69 124.46) (xy 104.14 124.46)
 		)
@@
 	(wire
 		(pts
-			(xy 62.23 160.02) (xy 154.94 160.02)
+			(xy 62.23 158.75) (xy 154.94 158.75)
 		)
 		(stroke
@@
 	)
 	(sheet
-		(at 43.18 154.94)
+		(at 43.18 153.67)
 		(size 19.05 16.51)
 		(fields_autoplaced yes)
@@
 		)
 		(property "Sheetname" "PowerSystemRover"
-			(at 43.18 154.2284 0)
+			(at 43.18 152.9584 0)
 			(effects
 				(font
@@
 		)
 		(property "Sheetfile" "PowerSystemRover.kicad_sch"
-			(at 43.18 172.0346 0)
+			(at 43.18 170.7646 0)
 			(effects
 				(font
@@
 		)
 		(property "Field2" ""
-			(at 43.18 154.94 0)
+			(at 43.18 153.67 0)
 			(effects
 				(font
@@
 				)
 				(hide yes)
+			)
+		)
+		(pin "Vout (5V)" output
+			(at 62.23 156.21 0)
+			(effects
+				(font
+					(size 1.27 1.27)
+				)
+				(justify right)
 			)
 		)
@@
 		)
 		(pin "Vout (4S - 14V)" output
-			(at 62.23 160.02 0)
-			(effects
-				(font
+			(at 62.23 158.75 0)
+			(effects
+				(font
