File: KiCad/Complete-Rover-Systems/PowerSystemRover.kicad_sch (KiCad schematic)
At the start: 1 part

Commit message: updated kicads
Parts:
- removed BT1: Battery, symbol Device:Battery
- added BT2: Battery, symbol Device:Battery
- added U13: Buck, Converter_DCDC:Converter_DCDC_Murata_OKI-78SR_Vertical, symbol Converter_DCDC:OKI-78SR-3.3_1.5-W36H-C
Connections:
- net GND: now also BT2.2 (-), U13.2 (GND)
- net Vout (4S - 14V): now also BT2.1 (+), U13.1 (IN)
- new net Vout (5V): U13.3 (OUT)
Changed lines of the file:
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@@
 	(generator_version "8.0")
 	(paper "A4")
-	(wire
-		(pts
-			(xy 87.63 106.68) (xy 132.08 106.68)
-		)
-		(stroke
-			(width 0)
-			(type default)
-		)
-	)
-	(wire
-		(pts
-			(xy 87.63 116.84) (xy 130.81 116.84)
+	(junction
+		(at 121.92 123.19)
+		(diameter 0)
+		(color 0 0 0 0)
+	)
+	(junction
+		(at 137.16 133.35)
+		(diameter 0)
+		(color 0 0 0 0)
+	)
+	(wire
+		(pts
+			(xy 137.16 133.35) (xy 156.21 133.35)
+		)
+		(stroke
+			(width 0)
+			(type default)
+		)
+	)
+	(wire
+		(pts
+			(xy 144.78 123.19) (xy 157.48 123.19)
+		)
+		(stroke
+			(width 0)
+			(type default)
+		)
+	)
+	(wire
+		(pts
+			(xy 121.92 116.84) (xy 121.92 123.19)
+		)
+		(stroke
+			(width 0)
+			(type default)
+		)
+	)
+	(wire
+		(pts
+			(xy 109.22 133.35) (xy 137.16 133.35)
+		)
+		(stroke
+			(width 0)
+			(type default)
+		)
+	)
+	(wire
+		(pts
+			(xy 109.22 123.19) (xy 121.92 123.19)
+		)
+		(stroke
+			(width 0)
+			(type default)
+		)
+	)
+	(wire
+		(pts
+			(xy 121.92 116.84) (xy 157.48 116.84)
+		)
+		(stroke
+			(width 0)
+			(type default)
+		)
+	)
+	(wire
+		(pts
+			(xy 137.16 130.81) (xy 137.16 133.35)
+		)
+		(stroke
+			(width 0)
+			(type default)
+		)
+	)
+	(wire
+		(pts
+			(xy 121.92 123.19) (xy 129.54 123.19)
 		)
 		(stroke
@@
 	)
 	(rectangle
-		(start 72.39 96.52)
-		(end 132.08 128.27)
+		(start 97.79 113.03)
+		(end 157.48 144.78)
 		(stroke
 			(width 0)
@@
 		)
 	)
-	(hierarchical_label "Vout (4S - 14V)"
-		(shape output)
-		(at 132.08 106.68 0)
+	(hierarchical_label "GND"
+		(shape input)
+		(at 156.21 133.35 0)
 		(fields_autoplaced yes)
 		(effects
@@
 		)
 	)
-	(hierarchical_label "GND"
-		(shape input)
-		(at 130.81 116.84 0)
+	(hierarchical_label "Vout (4S - 14V)"
+		(shape output)
+		(at 157.48 116.84 0)
 		(fields_autoplaced yes)
 		(effects
@@
 		)
 	)
+	(hierarchical_label "Vout (5V)"
+		(shape output)
+		(at 157.48 123.19 0)
+		(fields_autoplaced yes)
+		(effects
+			(font
+				(size 1.27 1.27)
+			)
+			(justify left)
+		)
+	)
 	(symbol
 		(lib_id "Device:Battery")
-		(at 87.63 111.76 0)
+		(at 109.22 128.27 0)
 		(unit 1)
 		(exclude_from_sim no)
@@
 		(dnp no)
 		(fields_autoplaced yes)
-		(property "Reference" "BT1"
-			(at 91.44 109.9184 0)
+		(property "Reference" "BT2"
+			(at 113.03 126.4284 0)
 			(effects
 				(font
@@
 		)
 		(property "Value" "Battery"
-			(at 91.44 112.4584 0)
+			(at 113.03 128.9684 0)
 			(effects
 				(font
@@
 		)
 		(property "Footprint" ""
-			(at 87.63 110.236 90)
+			(at 109.22 126.746 90)
 			(effects
 				(font
@@
 		)
 		(property "Datasheet" "~"
-			(at 87.63 110.236 90)
+			(at 109.22 126.746 90)
 			(effects
 				(font
@@
 		)
 		(property "Description" "Multiple-cell battery"
-			(at 87.63 111.76 0)
+			(at 109.22 128.27 0)
 			(effects
 				(font
@@
 			(project "Complete-Rover-Systems"
 				(path "/6fa62cff-8e96-404b-9f84-9cfa132ad8cc/6832115b-c53d-4fc5-8a54-f93fdadad37c"
-					(reference "BT1")
+					(reference "BT2")
 					(unit 1)
 				)
+			)
+		)
+	)
+	(symbol
+		(lib_id "Converter_DCDC:OKI-78SR-3.3_1.5-W36H-C")
+		(at 137.16 123.19 0)
+		(unit 1)
+		(exclude_from_sim no)
+		(in_bom yes)
+		(on_board yes)
+		(dnp no)
+		(fields_autoplaced yes)
+		(property "Reference" "U13"
+			(at 137.16 116.84 0)
+			(effects
+				(font
+					(size 1.27 1.27)
+				)
+			)
+		)
+		(property "Value" "Buck"
+			(at 137.16 119.38 0)
+			(effects
+				(font
+					(size 1.27 1.27)
+				)
+			)
+		)
+		(property "Footprint" "Converter_DCDC:Converter_DCDC_Murata_OKI-78SR_Vertical"
+			(at 138.43 129.54 0)
+			(effects
+				(font
+					(size 1.27 1.27)
+					(italic yes)
+				)
+				(justify left)
+				(hide yes)
+			)
+		)
+		(property "Datasheet" "https://power.murata.com/data/power/oki-78sr.pdf"
+			(at 137.16 123.19 0)
+			(effects
+				(font
+					(size 1.27 1.27)
+				)
+				(hide yes)
+			)
+		)
+		(property "Description" "1.5A Step-Down DC/DC-Regulator, 7-36V input, 3.3V fixed Output Voltage, LM78xx replacement, -40°C to +85°C, OKI-78SR_Horizontal"
+			(at 137.16 123.19 0)
+			(effects
+				(font
+					(size 1.27 1.27)
+				)
+				(hide yes)
+			)
+		)
+		(pin "1"
+		)
+		(pin "3"
+		)
+		(pin "2"
+		)
+		(instances
+			(project "Complete-Rover-Systems"
+				(path "/6fa62cff-8e96-404b-9f84-9cfa132ad8cc/6832115b-c53d-4fc5-8a54-f93fdadad37c"
+					(reference "U13")
+					(unit 1)
+				)
