File: KiCad/Complete-Drone-Systems/DronePower.kicad_sch (KiCad schematic)
At the start: 2 parts, among them U4 Buck

Commit message: updated kicad prints
Connections:
- net GND: no longer BT1.1 (+), U4.1 (IN)
- new net Vout (6S - 22.2V): BT1.1 (+), U4.1 (IN)
Changed lines of the file:
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@@
-		(color 0 0 0 0)
-	)
-	(junction
-		(at 129.54 107.95)
-		(diameter 0)
 		(color 0 0 0 0)
 	)
@@
 	(wire
 		(pts
-			(xy 129.54 97.79) (xy 129.54 107.95)
+			(xy 116.84 107.95) (xy 144.78 107.95)
 		)
 		(stroke
-			(width 0)
-			(type default)
-		)
-	)
-	(wire
-		(pts
-			(xy 129.54 107.95) (xy 144.78 107.95)
-		)
-		(stroke
-			(width 0)
-			(type default)
-		)
-	)
-	(wire
-		(pts
-			(xy 116.84 107.95) (xy 129.54 107.95)
-		)
-		(stroke
